Commit message: add scanner

File: fwis_simulation/urdf/fwis_effort.xacro.urdf (robot description, URDF)
Before this commit: robot mobile_assembly, 14 links, 13 joints
Links:
- removed link arucam_left_link
- removed link arucam_right_link
- added link scanner1_link, mass 0.380816890715382; collision mesh filename=file://$(find fwis_simulation)/models/mobile_assembly/meshe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 scale=1 1 1; visual mesh filename=file://$(find fwis_simulation)/models/mobile_assembly/meshe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 scale=1 1 1
- added link scanner2_link, mass 0.380816890715382; collision mesh filename=file://$(find fwis_simulation)/models/mobile_assembly/meshe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 scale=1 1 1; visual mesh filename=file://$(find fwis_simulation)/models/mobile_assembly/meshe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 scale=1 1 1
- link base_link: mass 11.0989219089157 -> 19.5136122526707
Joints:
- removed joint arucam_left_joint
- removed joint arucam_right_joint
- added joint scanner1_joint: type continuous, parent base_link, child scanner1_link, origin xyz=0.0271 0.0918 0.3976 rpy=0 0 0, axis 1 0 0, limit lower=-3.14 upper=3.14 effort=2.5 velocity=6.7
- added joint scanner2_joint: type continuous, parent base_link, child scanner2_link, origin xyz=-0.0271 -0.0918 0.3976 rpy=0 0 0, axis -1 0 0, limit lower=-3.14 upper=3.14 effort=2.5 velocity=6.7
- joint drive1_axis_joint: origin xyz=0.215 0.215 0.125675219801023 rpy=0 0 0 -> xyz=0.215 0.215 0.09 rpy=0 0 0
- joint drive2_axis_joint: origin xyz=0.215 -0.215 0.125675219801022 rpy=0 0 0 -> xyz=0.215 -0.215 0.09 rpy=0 0 0
- joint drive3_axis_joint: origin xyz=-0.215 0.215 0.125675219801014 rpy=0 0 0 -> xyz=-0.215 0.215 0.09 rpy=0 0 0
- joint drive4_axis_joint: origin xyz=-0.215 -0.215 0.125675219801014 rpy=0 0 0 -> xyz=-0.215 -0.215 0.09 rpy=0 0 0
- joint imu_joint: origin xyz=0 0 0.211175000000014 rpy=0 0 0 -> xyz=0 0 -0.0357 rpy=0 0 0
- joint lidar_joint: origin xyz=0 0 0 rpy=0 0 0 -> xyz=0 0 -0.0357 rpy=0 0 0
- joint motor3_axis_joint: origin xyz=0 -0.000199999999998729 -0.1 rpy=0 0 0 -> xyz=0 0 -0.1 rpy=0 0 0

File: fwis_simulation/urdf/fwis_position_velocity.xacro.urdf (robot description, URDF)
Before this commit: robot mobile_assembly, 14 links, 13 joints
Links:
- removed link arucam_left_link
- removed link arucam_right_link
- added link scanner1_link, mass 0.380816890715382; collision mesh filename=file://$(find fwis_simulation)/models/mobile_assembly/meshe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 scale=1 1 1; visual mesh filename=file://$(find fwis_simulation)/models/mobile_assembly/meshe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 scale=1 1 1
- added link scanner2_link, mass 0.380816890715382; collision mesh filename=file://$(find fwis_simulation)/models/mobile_assembly/meshe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 scale=1 1 1; visual mesh filename=file://$(find fwis_simulation)/models/mobile_assembly/meshe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 scale=1 1 1
- link base_link: mass 11.0989219089157 -> 19.5136122526707
Joints:
- removed joint arucam_left_joint
- removed joint arucam_right_joint
- added joint scanner1_joint: type continuous, parent base_link, child scanner1_link, origin xyz=0.0271 0.0918 0.3976 rpy=0 0 0, axis 1 0 0, limit lower=-3.14 upper=3.14 effort=2.5 velocity=6.7
- added joint scanner2_joint: type continuous, parent base_link, child scanner2_link, origin xyz=-0.0271 -0.0918 0.3976 rpy=0 0 0, axis -1 0 0, limit lower=-3.14 upper=3.14 effort=2.5 velocity=6.7
- joint drive1_axis_joint: origin xyz=0.215 0.215 0.125675219801023 rpy=0 0 0 -> xyz=0.215 0.215 0.09 rpy=0 0 0
- joint drive2_axis_joint: origin xyz=0.215 -0.215 0.125675219801022 rpy=0 0 0 -> xyz=0.215 -0.215 0.09 rpy=0 0 0
- joint drive3_axis_joint: origin xyz=-0.215 0.215 0.125675219801014 rpy=0 0 0 -> xyz=-0.215 0.215 0.09 rpy=0 0 0
- joint drive4_axis_joint: origin xyz=-0.215 -0.215 0.125675219801014 rpy=0 0 0 -> xyz=-0.215 -0.215 0.09 rpy=0 0 0
- joint imu_joint: origin xyz=0 0 0.211175000000014 rpy=0 0 0 -> xyz=0 0 -0.0357 rpy=0 0 0
- joint lidar_joint: origin xyz=0 0 0 rpy=0 0 0 -> xyz=0 0 -0.0357 rpy=0 0 0
- joint motor3_axis_joint: origin xyz=0 -0.000199999999998729 -0.1 rpy=0 0 0 -> xyz=0 0 -0.1 rpy=0 0 0

Commit message: add camera

File: fwis_simulation/urdf/fwis_effort.xacro.urdf (robot description, URDF)
Before this commit: robot mobile_assembly, 14 links, 13 joints
Links:
- added link camera_link, mass 0.0447532238450961; collision mesh filename=file://$(find fwis_simulation)/models/mobile_assembly/meshe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 scale=1 1 1; visual mesh filename=file://$(find fwis_simulation)/models/mobile_assembly/meshe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 scale=1 1 1
Joints:
- added joint camera_joint: type fixed, parent base_link, child camera_link, origin xyz=0.325 0 0.27 rpy=0 0 0

File: fwis_simulation/urdf/fwis_position_velocity.xacro.urdf (robot description, URDF)
Before this commit: robot mobile_assembly, 14 links, 13 joints
Links:
- added link camera_link, mass 0.0447532238450961; collision mesh filename=file://$(find fwis_simulation)/models/mobile_assembly/meshe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 scale=1 1 1; visual mesh filename=file://$(find fwis_simulation)/models/mobile_assembly/meshe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 scale=1 1 1
Joints:
- added joint camera_joint: type fixed, parent base_link, child camera_link, origin xyz=0.325 0 0.27 rpy=0 0 0
