Commit message: lidar rotation

File: fwis_robot/urdf/fwis_position_velocity.xacro.urdf (robot description, URDF)
Before this commit: robot mobile_assembly, 14 links, 13 joints
Links:
- removed link lidar_link
- added link laser_frame, mass 0.0853398661286776; collision mesh filename=file://$(find fwis_robot)/models/mobile_assembly/meshes/lid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 scale=1 1 1; visual mesh filename=file://$(find fwis_robot)/models/mobile_assembly/meshes/lid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 scale=1 1 1
Joints:
- joint lidar_joint: child lidar_link -> laser_frame; origin xyz=0 0 -0.0357 rpy=0 0 0 -> xyz=0 0 -0.0357 rpy=0 0 1.5708

Commit message: add: avoiding obstacles

File: fwis_robot/urdf/fwis_position_velocity.xacro.urdf (robot description, URDF)
Before this commit: robot mobile_assembly, 14 links, 13 joints
Joints:
- joint lidar_joint: origin xyz=0 0 -0.0357 rpy=0 0 1.5708 -> xyz=0 0 0 rpy=0 0 1.5708
